File: Esp32_Presence_Sensor_hw.kicad_pcb (KiCad board)
At the start: 2 copper layers, 25.4 x 34.2 mm, 32 parts, among them J1 USB_C_16P, J2 P_01x08-0.9, J3 P_01x08-0.9, SW1 SW_2x4x3.5, SW2 SW_2x4x3.5, U1 ESP32-C3, Y1 40MHz

Commit message: Block (220VAC, DS18B20, Resitor photo, relay, oled, RF 315Mhz)
Parts:
- added C10: 10uF, Capacitor_SMD:C_0603_1608Metric, F.Cu at (201.0, 114.1)
- added C17: 10uF/16V, Capacitor_SMD:C_0805_2012Metric_Pad1.18x1.45mm_HandSolder, F.Cu at (206.3, 108.3)
- added C18: 100nF, Capacitor_SMD:C_0402_1005Metric, F.Cu at (214.9, 103.6)
- added C19: 1nF/200, Capacitor_SMD:C_0805_2012Metric_Pad1.18x1.45mm_HandSolder, F.Cu at (215.2, 111.3)
- added C2: 10uF, Capacitor_SMD:C_0603_1608Metric, F.Cu at (185.9, 55.6)
- added C20: 100nF/50V, Capacitor_SMD:C_0805_2012Metric_Pad1.18x1.45mm_HandSolder, F.Cu at (206.3, 105.3)
- added C21: 4.7uF/400V, Capacitor_THT:CP_Radial_D8.0mm_P3.50mm, F.Cu at (244.3, 58.8)
- added C22: 1nF/200, Capacitor_SMD:C_0805_2012Metric_Pad1.18x1.45mm_HandSolder, F.Cu at (211.1, 108.3)
- added C23: 10uF, Capacitor_SMD:C_0603_1608Metric, F.Cu at (190.0, 55.6)
- added C24: 100nF, Capacitor_SMD:C_0402_1005Metric, F.Cu at (214.9, 105.6)
- added C25: 1nF/25V, Capacitor_SMD:C_0805_2012Metric_Pad1.18x1.45mm_HandSolder, F.Cu at (211.1, 105.3)
- added C26: 560uF/6.3V, Capacitor_THT:CP_Radial_D10.0mm_P5.00mm, F.Cu at (215.7, 93.8)
- added C27: 100nF/50V, Capacitor_SMD:C_0805_2012Metric_Pad1.18x1.45mm_HandSolder, F.Cu at (201.4, 96.2)
- added C28: 100nF, Capacitor_SMD:C_0805_2012Metric_Pad1.18x1.45mm_HandSolder, F.Cu at (206.2, 111.3)
- added C29: 10uF, Capacitor_SMD:C_0805_2012Metric_Pad1.18x1.45mm_HandSolder, F.Cu at (201.4, 111.3)
- added C30: 100nF, Capacitor_SMD:C_0402_1005Metric, F.Cu at (204.4, 113.8)
- added C31: 10uF, Capacitor_SMD:C_0805_2012Metric_Pad1.18x1.45mm_HandSolder, F.Cu at (215.9, 101.1)
- added C32: 100nF, Capacitor_SMD:C_0805_2012Metric_Pad1.18x1.45mm_HandSolder, F.Cu at (219.4, 81.6)
- added C33: 100nF, Capacitor_SMD:C_0402_1005Metric, F.Cu at (219.7, 100.6)
- added C34: 1uF, Capacitor_SMD:C_0402_1005Metric, F.Cu at (210.0, 110.8)
- added C35: 100nF, Capacitor_SMD:C_0402_1005Metric, F.Cu at (231.3, 87.7)
- added C9: 100nF, Capacitor_SMD:C_0402_1005Metric, F.Cu at (217.8, 103.6)
- added D1: MB10F, Package_TO_SOT_SMD:TO-269AA, F.Cu at (140.7, 140.2)
- added D2: 1N4148, Diode_SMD:D_SMA, F.Cu at (246.2, 65.9)
- added D3: RS1J, Diode_SMD:D_SMA, F.Cu at (254.9, 62.7)
- added D4: SR240, Diode_SMD:D_SMA, F.Cu at (238.1, 70.4)
- added D5: 1N4148, Diode_SMD:D_SMA, F.Cu at (238.1, 65.9)
- added J2: Screw_Terminal_01x04, TerminalBlock:TerminalBlock_bornier-4_P5.08mm, F.Cu at (109.0, 141.0)
- added K1: G5LE-1, Relay_THT:Relay_SPDT_Omron-G5LE-1, F.Cu at (97.3, 141.5)
- added L2: L_Ferrite, Inductor_SMD:L_0805_2012Metric_Pad1.05x1.20mm_HandSolder, F.Cu at (181.5, 55.8)
- added Q1: Q_NPN_BEC, Package_TO_SOT_SMD:SOT-23, F.Cu at (201.4, 106.0)
- added Q2: 2SC1815/HF, Package_TO_SOT_SMD:SOT-23, F.Cu at (207.4, 101.6)
- added R10: 3R6, Resistor_SMD:R_1206_3216Metric_Pad1.30x1.75mm_HandSolder, F.Cu at (226.0, 85.1)
- added R11: 22K, Resistor_SMD:R_1206_3216Metric_Pad1.30x1.75mm_HandSolder, F.Cu at (237.1, 80.5)
- added R12: 3K3, Resistor_SMD:R_1206_3216Metric_Pad1.30x1.75mm_HandSolder, F.Cu at (226.9, 81.8)
- added R13: 10k, Resistor_SMD:R_0402_1005Metric, F.Cu at (199.2, 55.4)
- added R14: 22K, Resistor_SMD:R_1206_3216Metric_Pad1.30x1.75mm_HandSolder, F.Cu at (226.9, 88.4)
- added R15: R_Photo, Lib_Mr_DH:R_photo, F.Cu at (237.1, 75.7)
- added R16: 10k, Resistor_SMD:R_0402_1005Metric, F.Cu at (210.9, 55.4)
- added R17: 2.2K, Resistor_SMD:R_0402_1005Metric, F.Cu at (202.2, 55.4)
- added R18: 220R, Resistor_SMD:R_0402_1005Metric, F.Cu at (231.8, 62.6)
- added R19: 0R, Resistor_SMD:R_0402_1005Metric, F.Cu at (205.1, 55.4)
- added R20: 0R, Resistor_SMD:R_0402_1005Metric, F.Cu at (237.6, 62.6)
- added R21: 220R, Resistor_SMD:R_0402_1005Metric, F.Cu at (196.3, 55.4)
- added R22: 220R, Resistor_SMD:R_0402_1005Metric, F.Cu at (193.4, 56.3)
- added R23: 220R, Resistor_SMD:R_0402_1005Metric, F.Cu at (231.3, 81.1)
- added R24: 330R, Resistor_SMD:R_0402_1005Metric, F.Cu at (208.0, 55.4)
- added R25: 1k, Resistor_SMD:R_0402_1005Metric, F.Cu at (234.7, 62.6)
- added R4: 3R3/1W, Resistor_THT:R_Axial_DIN0617_L17.0mm_D6.0mm_P5.08mm_Vertical, F.Cu at (134.2, 140.8)
- added R6: 1M, Resistor_SMD:R_1206_3216Metric_Pad1.30x1.75mm_HandSolder, F.Cu at (202.0, 101.2)
- added R7: 1M, Resistor_SMD:R_1206_3216Metric_Pad1.30x1.75mm_HandSolder, F.Cu at (226.9, 91.6)
- added R8: 1M, Resistor_SMD:R_1206_3216Metric_Pad1.30x1.75mm_HandSolder, F.Cu at (220.0, 85.1)
- added R9: 1M, Resistor_SMD:R_1206_3216Metric_Pad1.30x1.75mm_HandSolder, F.Cu at (231.9, 85.1)
- added U2: SYN470R, Lib_Mr_DH:SYN470R_RF315Mhz, F.Cu at (164.2, -14.1)
- added U3: LD2410, Lib_Mr_DH:LD2410, F.Cu at (79.1, 102.6)
- added U4: CR1510, Package_SO:PowerIntegrations_SO-8C, F.Cu at (263.8, 57.3)
- added U5: DS18B20, Lib_Mr_DH:TO-92-TO92127P495H2044-3, F.Cu at (245.4, 71.1)
- added U6: EE13-5V, Lib_Mr_DH:EE13_6_6, F.Cu at (135.6, 128.4)
- added U7: RT9193, Package_TO_SOT_SMD:SOT-23-5_HandSoldering, F.Cu at (207.8, 97.0)
- added U8: PC817, Package_DIP:SMDIP-4_W9.53mm, F.Cu at (205.6, 91.4)
- added U9: 2.2inch_TFT_ILI9341_SPI, Lib_Mr_DH:TFT_ILI9341_2.2INCH, F.Cu at (286.6, 91.6)
- moved C11 67.5 mm to (107.7, 11.1)
- moved C12 67.5 mm to (101.6, 4.50)
- moved C13 67.5 mm to (106.8, 4.50)
- moved C14 67.5 mm to (94.2, 3.88)
- moved C15 67.5 mm to (96.6, 2.55)
- moved C16 67.5 mm to (96.8, 6.60)
- moved C17 67.5 mm to (94.6, 20.8)
- moved C18 67.5 mm to (98.2, 15.3)
- moved C3 67.5 mm to (96.1, 9.55)
- moved C6 67.5 mm to (98.5, 10.2)
- moved C7 67.5 mm to (102.4, 14.9)
- moved C8 67.5 mm to (107.7, 12.1)
- moved J1 67.5 mm to (101.7, 24.1)
- moved J2 67.5 mm to (90.4, 2.30)
- moved J3 67.5 mm to (112.1, 2.27)
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Connections:
- J1 pad A4: VBUS -> +5V
- J1 pad A9: VBUS -> +5V
- J1 pad B4: VBUS -> +5V
- J1 pad B9: VBUS -> +5V
- U1 pad 10: IO5 -> U1TXD
- U1 pad 12: IO6 -> /LCD_SCL
- U1 pad 13: IO7 -> /LCD_MISO
- U1 pad 14: IO8 -> /LCD_CS0
- U1 pad 16: IO10 -> /RELAY
- U1 pad 4: IO0 -> /RF_Data
- U1 pad 5: IO1 -> /DS18B20_Data
- U1 pad 6: IO2 -> /R_Photo
- U1 pad 8: IO3 -> /LCD_MOSI
- U1 pad 9: IO4 -> U1RXD
Routing:
- net IO10: track 15.0 -> 0.00 mm
- net /RELAY: track 0.00 -> 15.0 mm
- net /RF_Data: track 0.00 -> 14.2 mm
- net IO0: track 14.2 -> 0.00 mm
- net IO5: track 13.8 -> 0.00 mm
- net U1TXD: track 0.00 -> 13.8 mm
- net IO6: track 13.2 -> 0.00 mm
- net /LCD_SCL: track 0.00 -> 13.2 mm
- net /DS18B20_Data: track 0.00 -> 12.7 mm
- net IO1: track 12.7 -> 0.00 mm
- net IO3: track 11.4 -> 0.00 mm
- net /LCD_MOSI: track 0.00 -> 11.4 mm
- net U1RXD: track 0.00 -> 11.1 mm
- net IO4: track 11.1 -> 0.00 mm
- net VBUS: vias 3 -> 0
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Other:
- outline, holes or cut-outs redrawn

Commit message: Xep block nguan 220VAC
Parts:
- C2, C23: footprint Capacitor_SMD:C_0603_1608Metric -> Capacitor_SMD:C_0805_2012Metric
- C24, C9: footprint Capacitor_SMD:C_0402_1005Metric -> Capacitor_SMD:C_0805_2012Metric
- C30, C33, C34, C35: footprint Capacitor_SMD:C_0402_1005Metric -> Capacitor_SMD:C_0805_2012Metric_Pad1.18x1.45mm_HandSolder
- R10, R9: footprint Resistor_SMD:R_1206_3216Metric_Pad1.30x1.75mm_HandSolder -> Resistor_SMD:R_0805_2012Metric
- R12: footprint Resistor_SMD:R_1206_3216Metric_Pad1.30x1.75mm_HandSolder -> Resistor_SMD:R_0805_2012Metric_Pad1.20x1.40mm_HandSolder
- R13: footprint Resistor_SMD:R_0402_1005Metric -> Resistor_SMD:R_0805_2012Metric
- R18, R19, R20, R21, R22, R23, R24, R25: footprint Resistor_SMD:R_0402_1005Metric -> Resistor_SMD:R_0805_2012Metric_Pad1.20x1.40mm_HandSolder
- moved C21 141.7 mm to (123.3, 132.6)
- moved U2 133.8 mm to (53.7, 61.4)
- moved D4 118.6 mm to (130.8, 120.9), turned to 180 degrees
- moved R15 89.3 mm to (154.1, 108.6)
- moved R24 87.2 mm to (170.9, 134.4), turned to -90 degrees
- moved C26 82.2 mm to (136.9, 117.3)
- moved R19 70.3 mm to (200.4, 125.5)
- moved C2 69.1 mm to (179.5, 124.5)
- moved C23 69.1 mm to (183.6, 124.5)
- moved L2 69.1 mm to (175.1, 124.6)
- moved R13 69.1 mm to (192.8, 124.2)
- moved R16 69.1 mm to (204.5, 124.2)
- moved R17 69.1 mm to (195.7, 124.2)
- moved R21 69.1 mm to (189.9, 124.2)
- moved R22 69.1 mm to (187.0, 125.1)
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Connections:
- U1 pad 12: /LCD_SCL -> unconnected-(U1-Pad12)
- U1 pad 13: /LCD_MISO -> unconnected-(U1-Pad13)
- U1 pad 14: /LCD_CS0 -> unconnected-(U1-Pad14)
- U1 pad 8: /LCD_MOSI -> unconnected-(U1-Pad8)
Routing:
- net IO10: track 0.00 -> 15.0 mm
- net /RELAY: track 15.0 -> 0.00 mm
- net IO0: track 0.00 -> 14.2 mm
- net /RF_Data: track 14.2 -> 0.00 mm
- net U1TXD: track 13.8 -> 0.00 mm
- net IO5: track 0.00 -> 13.8 mm
- net IO6: track 0.00 -> 13.2 mm
- net /LCD_SCL: track 13.2 -> 0.00 mm
- net IO1: track 0.00 -> 12.7 mm
- net /DS18B20_Data: track 12.7 -> 0.00 mm
- net IO3: track 0.00 -> 11.4 mm
- net /LCD_MOSI: track 11.4 -> 0.00 mm
- net U1RXD: track 11.1 -> 0.00 mm
- net IO4: track 0.00 -> 11.1 mm

Commit message: them bien tro
Parts:
- removed the C17 at (94.6, 20.8)
- removed the C18 at (98.2, 15.3)
- removed the J2 at (90.4, 2.30)
- removed LED1: LED_0603_B, LED_SMD:LED_0603_1608Metric
- removed PS1: IA0503S, Package_TO_SOT_SMD:SOT-23-5
- removed the R4 at (94.2, 12.7)
- removed the R6 at (107.6, 13.2)
- added C36: 100nF, Capacitor_SMD:C_0805_2012Metric, F.Cu at (114.8, 91.8)
- added C37: 100nF, Capacitor_SMD:C_0805_2012Metric, F.Cu at (120.1, 91.8)
- added D6: 1N4148, Diode_SMD:D_SMA, F.Cu at (108.1, 85.5)
- added J4: 0R, Resistor_SMD:R_0805_2012Metric_Pad1.20x1.40mm_HandSolder, F.Cu at (204.4, 37.3)
- added J5: 0R, Resistor_SMD:R_0805_2012Metric_Pad1.20x1.40mm_HandSolder, F.Cu at (220.6, 31.6)
- added J6: 0R, Resistor_SMD:R_0805_2012Metric_Pad1.20x1.40mm_HandSolder, F.Cu at (204.4, 40.3)
- added J7: 0R, Resistor_SMD:R_0805_2012Metric_Pad1.20x1.40mm_HandSolder, F.Cu at (209.1, 37.3)
- added J8: 0R, Resistor_SMD:R_0805_2012Metric_Pad1.20x1.40mm_HandSolder, F.Cu at (225.3, 28.7)
- added J9: Conn_01x03_Male, Connector_PinSocket_2.54mm:PinSocket_1x03_P2.54mm_Vertical, F.Cu at (74.1, 80.0)
- added Q1: 2SC1815/HF, Package_TO_SOT_SMD:SOT-23, F.Cu at (201.0, 139.9)
- added R26: 0R, Resistor_SMD:R_0805_2012Metric_Pad1.20x1.40mm_HandSolder, F.Cu at (260.5, 121.5)
- added RV1: RM065-103 10K, Potentiometer_THT:Potentiometer_Runtron_RM-065_Vertical, F.Cu at (107.7, 89.4)
- added RV2: RM065-103 10K, Potentiometer_THT:Potentiometer_Runtron_RM-065_Vertical, F.Cu at (122.2, 89.2)
- added V1: Vit, Lib_Mr_DH:Vit, F.Cu at (195.8, 140.5)
- added V2: Vit, Lib_Mr_DH:Vit, F.Cu at (190.3, 146.0)
- added V3: Vit, Lib_Mr_DH:Vit, F.Cu at (108.9, 132.9)
- added V4: Vit, Lib_Mr_DH:Vit, F.Cu at (139.5, 87.6)
- C10: footprint Capacitor_SMD:C_0603_1608Metric -> Capacitor_SMD:C_0805_2012Metric
- C14, C18: footprint Capacitor_SMD:C_0402_1005Metric -> Capacitor_SMD:C_0805_2012Metric
- C26: footprint Capacitor_THT:CP_Radial_D10.0mm_P5.00mm -> Capacitor_THT:CP_Radial_D6.3mm_P2.50mm
- J3: value P_01x08-0.9 -> 0R; footprint Connector_PinHeader_2.54mm:PinHeader_1x08_P2.54mm_Vertical -> Resistor_SMD:R_0805_2012Metric_Pad1.20x1.40mm_HandSolder
- R1, R16, R17, R2, R3: footprint Resistor_SMD:R_0402_1005Metric -> Resistor_SMD:R_0805_2012Metric
- R11: footprint Resistor_SMD:R_1206_3216Metric_Pad1.30x1.75mm_HandSolder -> Resistor_SMD:R_0805_2012Metric
- R12: footprint Resistor_SMD:R_0805_2012Metric_Pad1.20x1.40mm_HandSolder -> Resistor_SMD:R_0805_2012Metric
- R5: value 2k -> 0R; footprint Resistor_SMD:R_0402_1005Metric -> Resistor_SMD:R_0805_2012Metric_Pad1.20x1.40mm_HandSolder
- SW1, SW2: value SW_2x4x3.5 -> SW_3.5x6x2.5; footprint EOS:ST-1114A -> Button_Switch_SMD:SW_DIP_SPSTx01_Slide_6.7x4.1mm_W8.61mm_P2.54mm_LowProfile
- moved R5 182.9 mm to (265.7, 118.6), turned to 0 degrees
- moved U4 127.5 mm to (121.8, 125.0)
- moved R25 122.8 mm to (89.6, 119.3), turned to -90 degrees
- moved D5 119.4 mm to (97.6, 119.4), turned to 180 degrees
- moved D2 116.5 mm to (112.3, 125.8), turned to 90 degrees
- moved U5 114.1 mm to (108.3, 119.8)
- moved J3 107.7 mm to (213.9, 37.3)
- moved ANT1 106.2 mm to (87.1, 105.6), turned to 90 degrees
- moved C15 103.8 mm to (89.8, 106.1), turned to -90 degrees
- moved R20 102.2 mm to (108.5, 99.7)
- moved L1 101.3 mm to (91.8, 105.7), turned to 0 degrees
- moved C16 99.3 mm to (93.8, 105.9), turned to -90 degrees
- moved C1 99.0 mm to (91.3, 102.7), turned to -90 degrees
- moved C5 97.5 mm to (92.7, 102.7), turned to -90 degrees
- moved C12 97.1 mm to (91.7, 101.1), turned to 0 degrees
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Connections:
- C21 pad 2: GND -> Earth
- J1 pad A4: +5V -> Net-(J1-PadA4)
- J1 pad A9: +5V -> Net-(J1-PadA4)
- J1 pad B4: +5V -> Net-(J1-PadA4)
- J1 pad B9: +5V -> Net-(J1-PadA4)
- J3 pad 1: U0TXD -> /LCD_DC
- J3 pad 2: U0RXD -> /GPIO2
- R17 pad 2: Net-(Q1-Pad1) -> Net-(Q1-Pad3)
- R18 pad 1: Net-(Q1-Pad3) -> Net-(Q1-Pad2)
- R19 pad 1: /RELAY -> /LCD_BL
- R21 pad 1: Net-(Q1-Pad3) -> Net-(Q1-Pad2)
- R22 pad 1: Net-(Q1-Pad3) -> Net-(Q1-Pad2)
- R23 pad 1: Net-(Q1-Pad3) -> Net-(Q1-Pad2)
- R5 pad 1: Net-(LED1-Pad2) -> +3.3V
- R5 pad 2: IO7 -> /LCD_DC
- U1 pad 12: unconnected-(U1-Pad12) -> /LCD_SCL
- U1 pad 13: unconnected-(U1-Pad13) -> /LCD_MISO
- U1 pad 14: unconnected-(U1-Pad14) -> /LCD_MOSI
- U1 pad 16: /RELAY -> /LCD_BL
- U1 pad 4: /RF_Data -> /ADC1_CH0
- U1 pad 5: /DS18B20_Data -> /ADC1_CH1
- U1 pad 6: /R_Photo -> /GPIO2
- U1 pad 8: unconnected-(U1-Pad8) -> /LCD_CS0
Routing:
- net GND: track 168.5 -> 22.8 mm, vias 51 -> 45
- net +3V3: track 82.1 -> 12.1 mm, vias 6 -> 0
- net EN: track 34.3 -> 0.00 mm, vias 3 -> 0
- net VBUS: track 32.7 -> 0.00 mm
- net D+: track 26.3 -> 0.00 mm, vias 2 -> 0
- net D-: track 24.9 -> 0.00 mm, vias 3 -> 0
- net IO7: track 24.3 -> 0.00 mm, vias 2 -> 0
- net IO8: track 23.5 -> 0.00 mm
- net IO9: track 18.6 -> 0.00 mm, vias 2 -> 0
- net IO10: track 15.0 -> 0.00 mm
- net IO0: track 14.2 -> 0.00 mm
- net IO5: track 13.8 -> 0.00 mm
- net IO6: track 13.2 -> 0.00 mm
- net U0TXD: track 13.1 -> 0.00 mm
- net IO1: track 12.7 -> 0.00 mm
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- removed copper zone on B.Cu, net GND
- removed copper zone on F.Cu, net GND
Other:
- board size 25.4 x 34.2 mm -> 63.2 x 62 mm
- board text removed: "0"
- board text removed: "1"
- board text removed: "10"
- board text removed: "2"
- board text removed: "3"
- board text removed: "3V3"
- board text removed: "4"
- board text removed: "5"
- board text removed: "6"
- board text removed: "7"
- board text removed: "8"
- board text removed: "EN"
- board text removed: "GND"
- board text removed: "RST"
- board text removed: "RX"
- board text removed: "TX"
- board text removed: "VBUS"

Commit message: sap xep linh kien qua pcb
Parts:
- removed C33: 100nF, Capacitor_SMD:C_0805_2012Metric_Pad1.18x1.45mm_HandSolder
- removed L2: L_Ferrite, Inductor_SMD:L_0805_2012Metric_Pad1.05x1.20mm_HandSolder
- removed the Q1 at (167.8, 106.4)
- removed V3, V4: Vit, Lib_Mr_DH:Vit
- added C38: 100nF, Capacitor_SMD:C_0805_2012Metric, F.Cu at (122.0, 76.6)
- C11, C4, C6, C8: footprint Capacitor_SMD:C_0402_1005Metric -> Capacitor_SMD:C_0805_2012Metric
- C14: footprint Capacitor_SMD:C_0805_2012Metric -> Capacitor_SMD:C_0805_2012Metric_Pad1.18x1.45mm_HandSolder
- C3: footprint Capacitor_SMD:C_0603_1608Metric -> Capacitor_SMD:C_0805_2012Metric
- C34: value 1uF -> 10uF
- J3, J4, J5, J6, J7, J8: footprint Resistor_SMD:R_0805_2012Metric_Pad1.20x1.40mm_HandSolder -> Resistor_SMD:R_0805_2012Metric
- R3: footprint Resistor_SMD:R_0805_2012Metric -> Resistor_SMD:R_0805_2012Metric_Pad1.20x1.40mm_HandSolder
- U9: moved to B.Cu
- moved C35 137.8 mm to (139.3, 86.8), turned to -90 degrees
- moved R5 134.2 mm to (135.4, 86.8), turned to 90 degrees
- moved C34 133.4 mm to (141.4, 86.8), turned to -90 degrees
- moved U9 132.8 mm to (115.8, 128.4)
- moved R26 127.9 mm to (137.3, 86.8), turned to -90 degrees
- moved J8 115.8 mm to (126.3, 88.5), turned to 90 degrees
- moved J5 113.6 mm to (122.3, 88.5), turned to 90 degrees
- moved D3 102.7 mm to (134.3, 117.8), turned to 90 degrees
- moved J7 99.1 mm to (124.3, 88.5), turned to 90 degrees
- moved J3 98.1 mm to (130.2, 88.5), turned to 90 degrees
- moved J6 90.2 mm to (128.2, 88.5), turned to 90 degrees
- moved J4 88.5 mm to (132.2, 88.5), turned to 90 degrees
- moved Q1 74.4 mm to (151.5, 84.4), turned to 180 degrees
- moved V1 70.4 mm to (253.5, 100.2)
- moved V2 70.4 mm to (248.0, 105.7)
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Connections:
- C34 pad 1: Net-(C34-Pad1) -> +3.3V
- C35 pad 1: Net-(C34-Pad1) -> +3.3V
- U9 pad 10: Net-(C34-Pad1) -> +3.3V
- U9 pad 9: Net-(C34-Pad1) -> +3.3V
Routing:
- net +3V3: track 12.1 -> 5.34 mm
- net GND: track 22.8 -> 19.8 mm
- net VDD_SPI: track 1.73 -> 0.00 mm
Other:
- board size 63.2 x 62 mm -> 63.7 x 61.7 mm
- board text added: "LD2410"
- board text removed: "C3 Mini V1.0.0 WEMOS.CC"

Commit message: Ve xong PCB
Parts:
- added V3: Vit, Lib_Mr_DH:Vit, F.Cu at (93.1, 128.8)
- added V4: Vit, Lib_Mr_DH:Vit, F.Cu at (98.6, 134.3)
- C1, C12, C13, C15, C16, C5, C7: footprint Capacitor_SMD:C_0402_1005Metric -> Capacitor_SMD:C_0805_2012Metric
- J2: footprint TerminalBlock:TerminalBlock_bornier-4_P5.08mm -> TerminalBlock_Phoenix:TerminalBlock_Phoenix_MKDS-1,5-4-5.08_1x04_P5.08mm_Horizontal
- K1: footprint Relay_THT:Relay_SPDT_Omron-G5LE-1 -> Relay_THT:Relay_SPDT_SANYOU_SRD_Series_Form_C
- L1: footprint Inductor_SMD:L_0603_1608Metric -> Inductor_SMD:L_0805_2012Metric
- moved V1 157.6 mm to (98.6, 128.8)
- moved V2 157.6 mm to (93.1, 134.3)
- moved R18 5.79 mm to (151.4, 75.9)
- moved R23 5.79 mm to (151.4, 81.7)
- moved C7 2.79 mm to (125.6, 81.4), turned to 90 degrees
- moved C13 2.29 mm to (112.4, 77.1)
- moved D3 1.97 mm to (133.2, 116.1), turned to 180 degrees
- moved R21 1.96 mm to (151.4, 77.8)
- moved R22 1.91 mm to (151.4, 79.7)
- moved Y1 1.71 mm to (112.4, 80.2)
- moved C12 1.37 mm to (112.4, 83.3)
- moved R9 1.23 mm to (139.8, 116.3)
- moved C22 1.23 mm to (137.8, 116.1)
- moved C15 1.17 mm to (109.9, 90.0)
- moved R20 1.12 mm to (127.6, 93.9), turned to 180 degrees
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Connections:
- J2 pad 1: /L -> /Out_Lamp
- J2 pad 4: /Out_Lamp -> /L
- J9 pad 1: U0TXD -> U0RXD
- J9 pad 2: U0RXD -> U0TXD
- K1 pad 3: unconnected-(K1-Pad3) -> /Out_Lamp
- K1 pad 4: /Out_Lamp -> unconnected-(K1-Pad4)
Routing:
- net GND: track 19.8 -> 306.4 mm, vias 45 -> 91
- net +3V3: track 5.34 -> 192.5 mm, vias 0 -> 4
- net +5V: track 0.00 -> 137.5 mm, vias 0 -> 2
- net /L: track 0.00 -> 94.3 mm, vias 0 -> 11
- net Earth: track 0.00 -> 77.0 mm, vias 0 -> 2
- net /ADC_RV2: track 0.00 -> 53.9 mm, vias 0 -> 1
- net Net-(C21-Pad1): track 0.00 -> 52.3 mm, vias 0 -> 2
- net /LCD_BL: track 0.00 -> 49.1 mm, vias 0 -> 4
- net Net-(C19-Pad2): track 0.00 -> 45.5 mm, vias 0 -> 1
- net /Out_Lamp: track 0.00 -> 45.4 mm, vias 0 -> 6
- net /RF_Data: track 0.00 -> 42.6 mm, vias 0 -> 1
- net /ADC_RV1: track 0.00 -> 36.3 mm, vias 0 -> 2
- net D+: track 0.00 -> 31.2 mm, vias 0 -> 2
- net /LCD_CS0: track 0.00 -> 28.8 mm, vias 0 -> 2
- net D-: track 0.00 -> 28.5 mm, vias 0 -> 2
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- added copper zone on B.Cu, net GND
- added copper zone on F.Cu, net GND
Other:
- outline, holes or cut-outs redrawn
- board text added: "RF 315Mhz"
