File: Esp32_Presence_Sensor_hw.kicad_sch (KiCad schematic)
At the start: 32 parts, among them J1 USB_C_16P, J2 Conn_01x08_Male, J3 Conn_01x08_Male, SW1 SW_2x4x3.5, SW2 SW_2x4x3.5, U1 ESP32-C3, Y1 40MHz

Commit message: Block (220VAC, DS18B20, Resitor photo, relay, oled, RF 315Mhz)
Parts:
- removed J2, J3: Conn_01x08_Male, symbol Connector:Conn_01x08_Male
- added C10, C2, C23: 10uF, Capacitor_SMD:C_0603_1608Metric, symbol Device:C
- added C17: 10uF/16V, Capacitor_SMD:C_0805_2012Metric_Pad1.18x1.45mm_HandSolder, symbol Device:C
- added C18, C24, C30, C33, C35, C9: 100nF, Capacitor_SMD:C_0402_1005Metric, symbol Device:C
- added C19, C22: 1nF/200, Capacitor_SMD:C_0805_2012Metric_Pad1.18x1.45mm_HandSolder, symbol Device:C
- added C20, C27: 100nF/50V, Capacitor_SMD:C_0805_2012Metric_Pad1.18x1.45mm_HandSolder, symbol Device:C
- added C21: 4.7uF/400V, Capacitor_THT:CP_Radial_D8.0mm_P3.50mm, symbol Device:C_Polarized
- added C25: 1nF/25V, Capacitor_SMD:C_0805_2012Metric_Pad1.18x1.45mm_HandSolder, symbol Device:C
- added C26: 560uF/6.3V, Capacitor_THT:CP_Radial_D10.0mm_P5.00mm, symbol Device:C_Polarized
- added C34: 1uF, Capacitor_SMD:C_0402_1005Metric, symbol Device:C
- added D1: MB10F, Package_TO_SOT_SMD:TO-269AA, symbol Diode_Bridge:MB4S
- added D2, D5: 1N4148, Diode_SMD:D_SMA, symbol Diode:1N4148
- added D3: RS1J, Diode_SMD:D_SMA, symbol Diode:1N4148
- added D4: SR240, Diode_SMD:D_SMA, symbol Diode:NSR0340HT1G
- added J2: Screw_Terminal_01x04, TerminalBlock:TerminalBlock_bornier-4_P5.08mm, symbol Connector:Screw_Terminal_01x04
- added K1: G5LE-1, Relay_THT:Relay_SPDT_Omron-G5LE-1, symbol Relay:G5LE-1
- added L2: L_Ferrite, Inductor_SMD:L_0805_2012Metric_Pad1.05x1.20mm_HandSolder, symbol Device:L_Ferrite
- added Q1: Q_NPN_BEC, Package_TO_SOT_SMD:SOT-23, symbol Device:Q_NPN_BEC
- added Q2: 2SC1815/HF, Package_TO_SOT_SMD:SOT-23, symbol Transistor_BJT:2SC1815
- added R10: 3R6, Resistor_SMD:R_1206_3216Metric_Pad1.30x1.75mm_HandSolder, symbol Device:R
- added R11, R14: 22K, Resistor_SMD:R_1206_3216Metric_Pad1.30x1.75mm_HandSolder, symbol Device:R
- added R12: 3K3, Resistor_SMD:R_1206_3216Metric_Pad1.30x1.75mm_HandSolder, symbol Device:R
- added R13, R16: 10k, Resistor_SMD:R_0402_1005Metric, symbol Device:R
- added R15: R_Photo, Lib_Mr_DH:R_photo, symbol Device:R_Photo
- added R17: 2.2K, Resistor_SMD:R_0402_1005Metric, symbol Device:R
- added R18, R21, R22, R23: 220R, Resistor_SMD:R_0402_1005Metric, symbol Device:R
- added R19, R20: 0R, Resistor_SMD:R_0402_1005Metric, symbol Device:R
- added R24: 330R, Resistor_SMD:R_0402_1005Metric, symbol Device:R
- added R25: 1k, Resistor_SMD:R_0402_1005Metric, symbol Device:R
- added R4: 3R3/1W, Resistor_THT:R_Axial_DIN0617_L17.0mm_D6.0mm_P5.08mm_Vertical, symbol Device:R
- added R6, R7, R8, R9: 1M, Resistor_SMD:R_1206_3216Metric_Pad1.30x1.75mm_HandSolder, symbol Device:R
- added U2: SYN470R, Lib_Mr_DH:SYN470R_RF315Mhz, symbol Lib_Mr_DH:SYN470R
- added U3: LD2410, Lib_Mr_DH:LD2410, symbol Lib_Mr_DH:LD2410
- added U4: CR1510, Package_SO:PowerIntegrations_SO-8C, symbol Lib_Mr_DH:CR1510
- added U5: DS18B20, Lib_Mr_DH:TO-92-TO92127P495H2044-3, symbol Lib_Mr_DH:DS18B20
- added U6: EE13-5V, Lib_Mr_DH:EE13_6_6, symbol Lib_Mr_DH:EE13-5V
- added U8: PC817, Package_DIP:SMDIP-4_W9.53mm, symbol Isolator:PC817
- added U9: 2.2inch_TFT_ILI9341_SPI, Lib_Mr_DH:TFT_ILI9341_2.2INCH, symbol Lib_Mr_DH:2.2inch_TFT_ILI9341_SPI
- gave numbers to parts that had none: 5
Connections:
- net +3.3V: now also C33.1, L2.1
- net +3V3: now also C2.1, C23.1, C24.1, C9.1, R13.1, R15.1, U2.3 (VCC), U5.3 (VDD)
- net +5V: now also C10.1, C18.1, C26.1, C27.1, D4.1 (K), D5.1 (K), K1.5, R14.2, U3.1 (VCC), U8.4
- net GND: now also C10.2, C18.2, C2.2, C21.2, C23.2, C24.2, C26.2, C27.2, C30.2, C33.2, C34.2, C35.2, C9.2, Q1.2 (E), Q2.1 (E), R16.2, U2.6 (GND), U3.2 (GND), U5.1 (GND), U6.10, U8.2, U9.1 (GND), U9.2 (RESET), U9.8 (GND)
- net IO7: no longer U1.13 (MTDO/GPIO7)
- net U1RXD: now also U3.4 (TXD)
- net U1TXD: now also U3.3 (RXD)
- net IO0 renamed RF_Data
- net RF_Data: now also U2.4 (Data), U2.5 (Data)
- net IO1 renamed DS18B20_Data
- net DS18B20_Data: now also R13.2, U5.2 (DQ)
- net IO10 renamed RELAY
- net RELAY: now also R19.1
- net IO2 renamed R_Photo
- net R_Photo: now also C30.1, R15.2, R16.1
- net IO3 renamed LCD_MOSI
- net LCD_MOSI: now also U9.6 (SDA)
- net IO6 renamed LCD_SCL
- net LCD_SCL: now also U9.3 (SCL)
- net IO8 renamed LCD_CS0
- net LCD_CS0: now also U9.5 (CS)
- new net: D5.2 (A), K1.2, Q2.2 (C)
- new net: Q2.3 (B), R25.2
- new net: Q1.3 (C), R18.1, R21.1, R22.1, R23.1
- new net: R11.2, R12.1, U4.6 (Vsense)
- new net: C34.1, C35.1, L2.2, U9.10 (LEDA), U9.9 (VCC)
- new net: R25.1, U8.3
- new net: C21.1, C22.2, D1.3 (+), R6.1, R9.1, U6.1
- new net: D1.1, R4.1
- new net: R11.1, U6.5
- new net: C19.2, D2.2 (A), D3.2 (A), U4.1 (C), U4.2 (C), U6.2
- new net: C25.1, D4.2 (A), U6.6
- new net: C17.1, C19.1, C20.1, D2.1 (K), R8.2, U4.4 (VCC)
- new net: R10.1, U4.7 (Isense), U4.8 (E)
- new net: Q1.1 (B), R17.2
- new net: R6.2, R7.1
- new net: R7.2, R8.1
- new net: C22.1, D3.1 (K), R9.2
- new net: R24.2, U8.1
- new net: C25.2, R14.1
- new net: R19.2, R20.2, R24.1
- new net BL1-: R18.2, U9.11 (LEDK1)
- new net BL2-: R21.2, U9.12 (LEDK2)
- new net BL3-: R22.2, U9.13 (LEDK3)
- new net BL4-: R23.2, U9.14 (LEDK4)
- new net Earth: C17.2, C20.2, D1.4 (-), R10.2, R12.2, U4.5 (GND), U6.4
- new net L: D1.2, J2.1 (Pin_1), K1.1
- new net LCD_BL: R17.1
- new net LCD_DC: U9.4 (D/C)
- new net LCD_MISO: U1.13 (MTDO/GPIO7), U9.7 (SD0)
- new net LDOUT: R20.1, U3.5 (OUT)
- new net N: J2.2 (Pin_2), J2.3 (Pin_3), R4.2
- new net Out_Lamp: J2.4 (Pin_4), K1.4
- new net X+: U9.17 (XR)
- new net X-: U9.15 (XL)
- new net Y+: U9.18 (YD)
- new net Y-: U9.16 (YU)
- no-connect marks 8 -> 10
Other:
- note added: "Buton input"
- note added: "Convert 5VDC to 3.3VDC"
- note added: "DS18B20"
- note added: "ESP32-C3"
- note added: "GL5528"
- note added: "HLK-LD2410"
- note added: "Input: ~ 220VAC / 1.5A Output load: 220VAC / 10A"
- note added: "LCD 2.2Inch TFT-ILI9341"
- note added: "No conect"
- note added: "OFF"
- note added: "ON"
- note added: "RELAY"
- note added: "SYN470R RF315Mhz"
- note added: "USB"
- note added: "You can chose ctrl relay by ESP32 or LD2410"
- title: ESP32-C3 Sensor Human -> ESP32-C3 Rada Sensor
- moved on the sheet: ANT1, C1, C11, C12, C13, C14, C15, C16, C28, C29, C3, C31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

Commit message: them bien tro
Parts:
- removed LED1: LED_0603_B, LED_SMD:LED_0603_1608Metric, symbol Device:LED
- removed Q1: Q_NPN_BEC, Package_TO_SOT_SMD:SOT-23, symbol Device:Q_NPN_BEC
- added C36, C37: 100nF, Capacitor_SMD:C_0805_2012Metric, symbol Device:C
- added D6: 1N4148, Diode_SMD:D_SMA, symbol Device:D
- added J3, J4, J5, J6, J7, J8, R26: 0R, Resistor_SMD:R_0805_2012Metric_Pad1.20x1.40mm_HandSolder, symbol Device:R
- added J9: Conn_01x03_Male, Connector_PinSocket_2.54mm:PinSocket_1x03_P2.54mm_Vertical, symbol Connector:Conn_01x03_Male
- added Q1: 2SC1815/HF, Package_TO_SOT_SMD:SOT-23, symbol Transistor_BJT:2SC1815
- added RV1, RV2: RM065-103 10K, Potentiometer_THT:Potentiometer_Runtron_RM-065_Vertical, symbol Device:R_Potentiometer_Trim_US
- added V1, V2, V3, V4: Vit, Lib_Mr_DH:Vit, symbol Lib_Mr_DH:Vit
- C10, C2, C23: footprint Capacitor_SMD:C_0603_1608Metric -> Capacitor_SMD:C_0805_2012Metric
- C14, C18, C24, C9: footprint Capacitor_SMD:C_0402_1005Metric -> Capacitor_SMD:C_0805_2012Metric
- C26: footprint Capacitor_THT:CP_Radial_D10.0mm_P5.00mm -> Capacitor_THT:CP_Radial_D6.3mm_P2.50mm
- C30, C33, C34, C35: footprint Capacitor_SMD:C_0402_1005Metric -> Capacitor_SMD:C_0805_2012Metric_Pad1.18x1.45mm_HandSolder
- R1, R13, R16, R17, R2, R3: footprint Resistor_SMD:R_0402_1005Metric -> Resistor_SMD:R_0805_2012Metric
- R10, R11, R12, R9: footprint Resistor_SMD:R_1206_3216Metric_Pad1.30x1.75mm_HandSolder -> Resistor_SMD:R_0805_2012Metric
- R18, R19, R20, R21, R22, R23, R24, R25: footprint Resistor_SMD:R_0402_1005Metric -> Resistor_SMD:R_0805_2012Metric_Pad1.20x1.40mm_HandSolder
- R5: value 2k -> 0R; footprint Resistor_SMD:R_0402_1005Metric -> Resistor_SMD:R_0805_2012Metric_Pad1.20x1.40mm_HandSolder
- SW1, SW2: value SW_2x4x3.5 -> SW_3.5x6x2.5; footprint EOS:ST-1114A -> Button_Switch_SMD:SW_DIP_SPSTx01_Slide_6.7x4.1mm_W8.61mm_P2.54mm_LowProfile
Connections:
- net IO7 is gone; now on net LCD_DC: R5.2
- net RELAY is gone; now on net LCD_BL: R19.1, U1.16 (GPIO10)
- net +3.3V: now also R5.1
- net +3V3: now also RV1.1, RV2.1
- net +5V: now also D6.1 (K); no longer J1.A4 (VBUS), J1.A9 (VBUS), J1.B4 (VBUS), J1.B9 (VBUS)
- net DS18B20_Data: now also J6.1; no longer U1.5 (XTAL_32K_N/ADC1_CH1)
- net Earth: now also C21.2
- net GND: now also C36.2, C37.2, J9.3 (Pin_3), Q1.1 (E), R26.2, RV1.3, RV2.3; no longer C21.2
- net LCD_CS0: now also U1.8 (GPIO3/ADC1_CH3), R26.1; no longer U1.14 (GPIO8)
- net LCD_DC: now also J3.1
- net LCD_MOSI: now also U1.14 (GPIO8); no longer U1.8 (GPIO3/ADC1_CH3)
- net RF_Data: now also J5.1; no longer U1.4 (XTAL_32K_P/ADC1_CH0)
- net R_Photo: now also J4.1; no longer U1.6 (GPIO2/ADC1_CH2)
- net U0RXD: now also J9.2 (Pin_2)
- net U0TXD: now also J9.1 (Pin_1)
- net at R18.1, R21.1, R22.1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: now also Q1.2 (C)
- net at R17.2: now also Q1.3 (B)
- new net: D6.2 (A), J1.A4 (VBUS), J1.A9 (VBUS), J1.B4 (VBUS), J1.B9 (VBUS)
- new net ADC1_CH0: J5.2, J7.2, U1.4 (XTAL_32K_P/ADC1_CH0)
- new net ADC1_CH1: J6.2, J8.2, U1.5 (XTAL_32K_N/ADC1_CH1)
- new net ADC_RV1: C36.1, J8.1, RV1.2
- new net ADC_RV2: C37.1, J7.1, RV2.2
- new net GPIO2: J3.2, J4.2, U1.6 (GPIO2/ADC1_CH2)
Other:
- moved on the sheet: ANT1, C1, C11, C12, C13, C14, C15, C16, C2, C3, C4, C5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

Commit message: sap xep linh kien qua pcb
Parts:
- removed C33: 100nF, Capacitor_SMD:C_0805_2012Metric_Pad1.18x1.45mm_HandSolder, symbol Device:C
- removed L2: L_Ferrite, Inductor_SMD:L_0805_2012Metric_Pad1.05x1.20mm_HandSolder, symbol Device:L_Ferrite
- added C38: 100nF, Capacitor_SMD:C_0805_2012Metric, symbol Device:C
- C11, C4, C6, C8: footprint Capacitor_SMD:C_0402_1005Metric -> Capacitor_SMD:C_0805_2012Metric
- C14: footprint Capacitor_SMD:C_0805_2012Metric -> Capacitor_SMD:C_0805_2012Metric_Pad1.18x1.45mm_HandSolder
- C3: footprint Capacitor_SMD:C_0603_1608Metric -> Capacitor_SMD:C_0805_2012Metric
- C34: value 1uF -> 10uF
- J3, J4, J5, J6, J7, J8: footprint Resistor_SMD:R_0805_2012Metric_Pad1.20x1.40mm_HandSolder -> Resistor_SMD:R_0805_2012Metric
- R3: footprint Resistor_SMD:R_0805_2012Metric -> Resistor_SMD:R_0805_2012Metric_Pad1.20x1.40mm_HandSolder
Connections:
- net +3.3V: now also C34.1, C35.1, U9.10 (LEDA), U9.9 (VCC)
- net GND: now also C38.2
- net IO9: now also C38.1
Other:
- moved on the sheet: SW2

Commit message: Ve xong PCB
Parts:
- C1, C12, C13, C15, C16, C5, C7: footprint Capacitor_SMD:C_0402_1005Metric -> Capacitor_SMD:C_0805_2012Metric
- J2: footprint TerminalBlock:TerminalBlock_bornier-4_P5.08mm -> TerminalBlock_Phoenix:TerminalBlock_Phoenix_MKDS-1,5-4-5.08_1x04_P5.08mm_Horizontal
- K1: footprint Relay_THT:Relay_SPDT_Omron-G5LE-1 -> Relay_THT:Relay_SPDT_SANYOU_SRD_Series_Form_C
- L1: footprint Inductor_SMD:L_0603_1608Metric -> Inductor_SMD:L_0805_2012Metric
Connections:
- net L: now also J2.4 (Pin_4); no longer J2.1 (Pin_1)
- net Out_Lamp: now also J2.1 (Pin_1), K1.3; no longer J2.4 (Pin_4), K1.4
- net U0RXD: now also J9.1 (Pin_1); no longer J9.2 (Pin_2)
- net U0TXD: now also J9.2 (Pin_2); no longer J9.1 (Pin_1)
Other:
- moved on the sheet: J2

Commit message: modified block LCD (sch & pcb)
Parts:
- removed R26, R5: 0R, Resistor_SMD:R_0805_2012Metric_Pad1.20x1.40mm_HandSolder, symbol Device:R
- removed V1, V2, V3, V4: Vit, Lib_Mr_DH:Vit, symbol Lib_Mr_DH:Vit
Connections:
- net GND: now also R17.1
- net LCD_BL renamed RELAY
- net RELAY: no longer R17.1
Other:
- moved on the sheet: Q1, R17, R18, R21, R22, R23
